File: playback/ch32v006_hardware/badapple006.kicad_pcb (KiCad board)
At the start: 2 copper layers, 16.4 x 16.2 mm, 34 parts, among them J1 OLED, J10 SCL, J11 SDA, J2 USB_C_Receptacle_USB2.0, J3 PG, J4 3v3, J5 GND, J6 RFO, J7 RFA, J8 APPLE, J9 RFO2, U1 CH32V006F8U6, U2 RS3236-3.3YUTDN4, Y1 24MHz

Commit message: bump playback + Schematic
Parts:
- added C12: 4.7u10v, Capacitor_SMD:C_0402_1005Metric, F.Cu at (74.4, 88.3)
- C1: value 2.2u16v -> 4.7u10v
- J4: value 3v3 -> 3.3
- R5: value 30 -> 49.9
- moved J3 0.40 mm to (74.6, 89.3)
- moved C7 0.34 mm to (71.2, 94.3)
- moved U1 0.21 mm to (72.9, 91.5)
- moved J8 0.12 mm to (74.0, 94.5)
- moved R4 0.07 mm to (72.3, 87.3)
- moved D1 0.06 mm to (71.1, 85.1)
- moved J6 0.06 mm to (71.8, 88.7)
Connections:
- J2 pad A8: SBU -> Net-(J2-SBU1)
- J2 pad B8: SBU -> Net-(J2-SBU1)
Routing:
- net SBU: track 10.3 -> 1.63 mm, vias 2 -> 0
- net Net-(J2-SBU1): track 0.00 -> 7.64 mm, vias 0 -> 2
- net GND: track 38.2 -> 38.9 mm
- net SWIO: track 1.90 -> 1.28 mm
Other:
- board text added: "badapple006 flip rev B(ad)"
- board text removed: "badapple006 flip rev B"
