File: playback/ch32v006_hardware/badapple006.kicad_sch (KiCad schematic)
At the start: 34 parts, among them J1 OLED, J10 SCL, J11 SDA, J2 USB_C_Receptacle_USB2.0, J3 PG, J4 3v3, J5 GND, J6 RFO, J7 RFA, J8 APPLE, J9 RFO2, U1 CH32V006F8U6, U2 RS3236-3.3YUTDN4, Y1 24MHz

Commit message: bump playback + Schematic
Parts:
- added C12: 10u6.3v, Capacitor_SMD:C_0402_1005Metric, symbol Device:C
Connections:
- net SBU: now also C12.1; no longer J2.A8 (SBU1), J2.B8 (SBU2)
- new net: C12.2, J2.A8 (SBU1), J2.B8 (SBU2)
Other:
- note removed: "Warning: OVCC's C2 bypass should operate at 7.9V. At 7.9V, C2's capacitance is rated at -80% We should consider trying to use a 0603 cap here."
- moved on the sheet: C6, U2
