File: hardware/badapple006.kicad_sch (KiCad schematic)
At the start: 35 parts, among them J10 5V, J11 GND, J12 RB066-6448-TSWHG01, J2 USB_C_Receptacle_USB2.0, J3 PG, J4 3v3, J5 GND, J6 RFO, J7 RFA, J8 APPLE, J9 RFO2, U1 CH32V006F8U7, U2 XC6206P332, Y1 24MHz

Commit message: Update to what was really orderedo
Parts:
- C11, C17, C4, C6: footprint Capacitor_SMD:C_0402_1005Metric -> Capacitor_SMD:C_0603_1608Metric; LCSC C23733 -> C19666
- J2: LCSC C2765186 -> C23376537
- U2: value XC6206P332 -> XC6206P362; LCSC C5446 -> C50593818
Other:
- note added: "VDD = 3.6V"
Changed lines of the file:
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@@
 		)
 	)
+	(text "VDD = 3.6V"
+		(exclude_from_sim no)
+		(at 205.232 64.008 0)
+		(effects
+			(font
+				(size 1.27 1.27)
+			)
+			(justify left bottom)
+		)
+	)
 	(text "OLED DISPLAY: RB066-6448-TSWHG01 (Ronboe)\nTell Agatha CNLohr sent you."
 		(exclude_from_sim no)
@@
 			)
 		)
-		(property "Footprint" "Capacitor_SMD:C_0402_1005Metric"
+		(property "Footprint" "Capacitor_SMD:C_0603_1608Metric"
 			(at 59.3852 55.88 0)
 			(hide yes)
@@
 			)
 		)
-		(property "LCSC" "C23733"
+		(property "LCSC" "C19666"
 			(at 58.42 52.07 0)
 			(hide yes)
@@
 			)
 		)
-		(property "Footprint" "Capacitor_SMD:C_0402_1005Metric"
+		(property "Footprint" "Capacitor_SMD:C_0603_1608Metric"
 			(at 155.9052 123.19 0)
 			(hide yes)
@@
 			)
 		)
-		(property "LCSC" "C23733"
+		(property "LCSC" "C19666"
 			(at 154.94 119.38 0)
 			(hide yes)
@@
 			)
 		)
-		(property "Value" "XC6206P332"
+		(property "Value" "XC6206P362"
 			(at 234.95 34.29 0)
 			(show_name no)
@@
 			)
 		)
-		(property "LCSC" "C5446"
+		(property "LCSC" "C50593818"
 			(at 234.95 38.1 0)
 			(hide yes)
@@
 			)
 		)
-		(property "Footprint" "Capacitor_SMD:C_0402_1005Metric"
+		(property "Footprint" "Capacitor_SMD:C_0603_1608Metric"
 			(at 182.5752 123.19 0)
 			(hide yes)
@@
 			)
 		)
-		(property "LCSC" "C23733"
+		(property "LCSC" "C19666"
 			(at 181.61 119.38 0)
 			(hide yes)
@@
 			)
 		)
-		(property "Footprint" "Capacitor_SMD:C_0402_1005Metric"
+		(property "Footprint" "Capacitor_SMD:C_0603_1608Metric"
 			(at 122.8852 152.4 0)
 			(hide yes)
@@
 			)
 		)
-		(property "LCSC" "C23733"
+		(property "LCSC" "C19666"
 			(at 121.92 148.59 0)
 			(hide yes)
@@
 			)
 		)
-		(property "LCSC" "C2765186"
+		(property "LCSC" "C23376537"
 			(at 53.34 135.89 0)
 			(hide yes)
