File: hardware/badapple006.kicad_pcb (KiCad board)
At the start: 2 copper layers, 16.5 x 16.2 mm, 35 parts, among them J10 5V, J11 GND, J12 RB066-6448-TSWHG01, J2 USB_C_Receptacle_USB2.0, J3 PG, J4 3v3, J5 GND, J6 RFO, J7 RFA, J8 APPLE, J9 RFO2, U1 CH32V006F8U7, U2 XC6206P362, Y1 24MHz

Commit message: Fixup wood layer
Other:
- board text added: "User.7 is laser cut for 1.8mm Thick Wood brace board"

Commit message: Update breakout and wood shim
Other:
- board text added: "User.3 is laser cut for 1.8mm Thick Wood brace board"
- board text removed: "User.7 is laser cut for 1.8mm Thick Wood brace board"
