File: hardware/sao/badapple006sao.kicad_pcb (KiCad board)
At the start: 2 copper layers, 16.5 x 16.2 mm, 31 parts, among them J1 SAO, J10 RFO2, J11 GND, J12 RB066-6448-TSWHG01, J13 GND, J3 PG, J4 3v3, J5 GND, J6 RFO, J7 RFA, J8 APPLE, J9 RFO2, U1 CH32V006F8U7, Y1 24MHz

Commit message: Update project, with slight echo for audio
Parts:
- removed C12: 10u6.3v, Capacitor_SMD:C_0402_1005Metric
- removed C8: 100n, Capacitor_SMD:C_0402_1005Metric
- added C15: 22u, Capacitor_SMD:C_0603_1608Metric, F.Cu at (71.6, 82.8)
- added C19: 22u, Capacitor_SMD:C_0603_1608Metric, F.Cu at (71.6, 84.3)
- added C20: 22u, Capacitor_SMD:C_0603_1608Metric, F.Cu at (71.6, 85.7)
- added C22: 22u, Capacitor_SMD:C_0603_1608Metric, F.Cu at (84.7, 85.5)
- J11: value GND -> VDD
- J7: value RFA -> GND
- moved J7 13.2 mm to (84.3, 83.4)
- moved C17 3.40 mm to (80.3, 89.2), turned to 180 degrees
- moved R5 2.63 mm to (85.7, 89.7)
- moved J10 2.61 mm to (71.2, 83.5)
- moved C10 2.34 mm to (84.1, 95.5), turned to 180 degrees
- moved Y1 1.71 mm to (83.6, 93.2)
- moved C16 1.22 mm to (80.9, 93.2), turned to -90 degrees
- moved C11 1.16 mm to (83.0, 91.2)
- moved R1 1.14 mm to (82.0, 87.6)
- moved C13 0.98 mm to (72.0, 87.1), turned to 180 degrees
- moved C18 0.92 mm to (82.7, 88.7)
- moved C9 0.45 mm to (85.5, 92.3)
- moved U1 0.33 mm to (77.6, 92.3)
- moved C14 0.12 mm to (72.1, 88.5)
- moved J9 0.11 mm to (76.5, 92.1)
Connections:
- C10 pad 2: Net-(U1-PA1/T1/T2/OPN0/XI/A1) -> Net-(U1-PA2/T1/T2/U2TX_/OPP0/X0A0)
- C9 pad 2: Net-(U1-PA2/T1/T2/U2TX_/OPP0/X0A0) -> Net-(U1-PA1/T1/T2/OPN0/XI/A1)
- J11 pad 1: GND -> OVDD
- J7 pad 1: Net-(J7-Pin_1) -> GND
- Y1 pad 1: Net-(U1-PA2/T1/T2/U2TX_/OPP0/X0A0) -> Net-(U1-PA1/T1/T2/OPN0/XI/A1)
- Y1 pad 3: Net-(U1-PA1/T1/T2/OPN0/XI/A1) -> Net-(U1-PA2/T1/T2/U2TX_/OPP0/X0A0)
Routing:
- net SBU: track 1.73 -> 20.2 mm, vias 0 -> 2
- net Net-(J10-Pin_1): track 15.0 -> 3.10 mm, vias 3 -> 1
- net GND: track 92.8 -> 81.1 mm
- net OVDD: track 41.9 -> 52.2 mm, vias 7 -> 8
- net Net-(U1-PA1/T1/T2/OPN0/XI/A1): track 5.65 -> 9.60 mm, vias 0 -> 2
- net Net-(D2-A): track 1.14 -> 3.98 mm
- net (no net): track 5.12 -> 2.56 mm
- net Net-(J12-Pin_14): track 4.93 -> 2.57 mm
- net Net-(J12-Pin_1): track 3.80 -> 1.87 mm
- net Net-(U1-PA2/T1/T2/U2TX_/OPP0/X0A0): track 9.26 -> 7.69 mm, vias 2 -> 0
- net DPU: track 1.33 -> 0.00 mm
- net REDCOLOR: track 18.2 -> 17.0 mm
- net SWIO: track 17.9 -> 16.8 mm
- net Net-(J12-Pin_13): track 5.01 -> 4.09 mm
- net Net-(J7-Pin_1): track 0.61 -> 0.00 mm, vias 1 -> 0
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Other:
- outline, holes or cut-outs redrawn
- board text added: "+"
- board text added: "1.6mm Thick Red FR4 OSP Coating 4x5 Array"
- board text added: "AUD+"
- board text added: "PG"
- board text added: "rev b"
- board text removed: "rev -"
