File: hardware/sao/badapple006sao.kicad_sch (KiCad schematic)
At the start: 31 parts, among them J1 SAO, J10 RFO2, J11 GND, J12 RB066-6448-TSWHG01, J13 GND, J3 PG, J4 3v3, J5 GND, J6 RFO, J7 RFA, J8 APPLE, J9 RFO2, U1 CH32V006F8U7, Y1 24MHz

Commit message: Update project, with slight echo for audio
Parts:
- removed C12: 10u6.3v, Capacitor_SMD:C_0402_1005Metric, symbol Device:C
- removed C8: 100n, Capacitor_SMD:C_0402_1005Metric, symbol Device:C
- added C15, C19, C20, C22: 22u, Capacitor_SMD:C_0603_1608Metric, symbol Device:C
- J11: value GND -> VDD
- J7: value RFA -> GND
Connections:
- net GND: now also J7.1 (Pin_1), C22.2; no longer J11.1 (Pin_1)
- net SBU: now also C15.2, C19.2, C20.2
- net VDD: now also J11.1 (Pin_1), C22.1
- net at J10.1 (Pin_1): now also C15.1, C19.1, C20.1
- net at C9.2, Y1.1: now also U1.2 (PA1/T1/T2/OPN0/XI/A1); no longer U1.3 (PA2/T1/T2/U2TX_/OPP0/X0A0)
- net at C10.2, Y1.3: now also U1.3 (PA2/T1/T2/U2TX_/OPP0/X0A0); no longer U1.2 (PA1/T1/T2/OPN0/XI/A1)
Other:
- moved on the sheet: J10
