File: hardware/usbc_headphone_breakout/usbc_headphone_breakout.kicad_pcb (KiCad board)
At the start: 2 copper layers, 24 x 17.7 mm, 6 parts, among them J1 USB_C_Receptacle_USB2.0_16P, J2 USB_C_Plug, J4 AudioJack3_Ground

Commit message: Update breakout and wood shim
Parts:
- removed ?: , 
- J4: footprint Connector_Audio:Jack_3.5mm_CUI_SJ-3524-SMT_Horizontal -> cnhardware:Jack_3.5mm_MINI_BackMount_SOFNG_PJ-320B
- moved J1 1.00 mm to (114.8, 82.3)
Connections:
- C1 pad 1: Net-(J2-SBU1) -> Net-(J2-SBU2)
- C2 pad 1: Net-(J2-SBU2) -> Net-(J2-SBU1)
- J1 pad S1: GND -> (no net)
- J2 pad A5: Net-(J1-CC1) -> Net-(J2-SBU1)
- J2 pad A8: Net-(J2-SBU1) -> Net-(J1-CC2)
- J2 pad B5: Net-(J1-CC2) -> Net-(J2-SBU2)
- J2 pad B8: Net-(J2-SBU2) -> Net-(J1-CC1)
Routing:
- net GND: track 45.9 -> 23.9 mm, vias 15 -> 14
- net Net-(J2-SBU1): track 6.93 -> 14.3 mm
- net Net-(J2-SBU2): track 14.6 -> 7.33 mm
- net Net-(C1-Pad2): track 4.74 -> 0.93 mm
- net Net-(J1-VBUS-PadA4): track 28.5 -> 25.0 mm
- net Net-(J1-CC1): track 8.29 -> 5.87 mm, vias 0 -> 1
- net Net-(J1-D--PadA7): track 11.8 -> 10.9 mm, vias 2 -> 3
- net Net-(J1-CC2): track 9.45 -> 9.08 mm, vias 1 -> 0
- net Net-(J1-D+-PadA6): track 10.9 -> 10.8 mm, vias 2 -> 0
Other:
- board size 24 x 17.7 mm -> 23 x 17.7 mm
- board text added: "badderapple usbc headphone breakout rev A"
- board text removed: "badderapple usbc headphone breakout rev -"

Commit message: Update with fixed flip of D+/D-
Connections:
- J2 pad A6: Net-(J1-D+-PadA6) -> Net-(J1-D--PadA7)
- J2 pad A7: Net-(J1-D--PadA7) -> Net-(J1-D+-PadA6)
Routing:
- net Net-(J1-D--PadA7): track 10.9 -> 10.3 mm, vias 3 -> 2
Other:
- board text added: "badderapple usbc headphone breakout rev B"
- board text removed: "badderapple usbc headphone breakout rev A"
